Commit message: Robot modeling - Add the rear wheel

File: src/box_bot_description/urdf/box_bot.urdf (robot description, URDF)
Before this commit: robot box_bot, 5 links, 4 joints
Links:
- added link rear_caster_wheel, mass 0.1; collision sphere radius=0.05; visual sphere radius=0.05
Joints:
- added joint rear_caster_wheel_joint: type fixed, parent base_link, child rear_caster_wheel, origin xyz=-0.2 0 -0.1

Commit message: Add base_footprint and attached abse_link to it - Update DiffDrive plugin
Remove joint_state_publisher to avoid conflict with Bridge:

File: src/box_bot_description/urdf/box_bot.urdf (robot description, URDF)
Before this commit: robot box_bot, 6 links, 5 joints
Links:
- added link base_footprint
Joints:
- added joint base_joint: type fixed, parent base_footprint, child base_link, origin xyz=0 0 0.15 rpy=0 0 0
